Commit message: basic sim

File: description/robot.urdf.xacro (robot description, xacro)
@@ -2,3 +2,4 @@
 <robot xmlns:xacro="http://www.ros.org/wiki/xacro"  name="robot">
     <xacro:include filename="robot_core_new.xacro" />
+    <xacro:include filename="gazebo_control.xacro"/>
 </robot>

File: description/robot_core_new.xacro (robot description, xacro)
@@ -21,5 +21,5 @@
         <parent link="base_link"/>
         <child link="chassis"/>
-        <origin xyz="-0.275 0 0"/>  <!-- origin behind bse link -->
+        <origin xyz="-0.275 0 0"/>  <!-- origin behind base link -->
     </joint>
     <link name="chassis">
@@ -37,8 +37,11 @@
             </geometry>
         </collision>
-        <xacro:inertial_box mass="25" x="0.34" y="0.34" z="0.725">
+        <xacro:inertial_box mass="0.5" x="0.34" y="0.34" z="0.725">
             <origin xyz="0.17 0 0.3625" rpy="0 0 0"/>
         </xacro:inertial_box>
     </link>
+    <gazebo reference = "chassis">
+        <material>Gazebo/White</material>
+    </gazebo>
     <!-- LEFT WHEEL LINK -->
     <joint name="left_wheel_joint" type="continuous">
@@ -64,6 +67,9 @@
         </xacro:inertial_cylinder>
     </link>
+    <gazebo reference="left_wheel">
+        <material>Gazebo/Blue</material>
+    </gazebo>
     <!-- RIGHT WHEEL LINK -->
-    <joint name="rightwheel_joint" type="continuous">
+    <joint name="right_wheel_joint" type="continuous">
         <parent link="base_link"/>
         <child link="right_wheel"/>
@@ -87,4 +93,7 @@
         </xacro:inertial_cylinder>
     </link>
+    <gazebo reference="right_wheel">
+        <material>Gazebo/Blue</material>
+    </gazebo>
     <!-- CASTER WHEEL LINK -->
     <joint name="caster_wheel_joint" type="fixed">
@@ -109,3 +118,8 @@
         </xacro:inertial_sphere>
     </link>
+    <gazebo reference="caster_wheel">
+        <material>Gazebo/Black</material>
+        <mu1 value="0.001"/>
+        <mu2 value="0.001"/>
+    </gazebo>
 </robot>

Commit message: -

File: description/robot.urdf.xacro (robot description, xacro)
@@ -5,3 +5,4 @@
     <!-- <xacro:include filename="camera.xacro"/> -->
     <xacro:include filename="depth_camera.xacro"/>
+    <xacro:include filename="lidar.xacro"/>
 </robot>

File: description/robot_core_new.xacro (robot description, xacro)
@@ -13,4 +13,7 @@
     <material name="black">
         <color rgba="0 0 0 1"/>
+    </material>
+    <material name="red">
+        <color rgba="1 0 0 1"/>
     </material>
     <!-- BASE LINK -->
@@ -32,11 +35,11 @@
         </visual>
         <collision>  <!-- สร้างแบบจำลองที่เห็นในโปรแกรม -->
-            <origin xyz="0.17 0 0.3625"/>  <!-- ตั้ง origin ใหม่ -->
+            <origin xyz="0.17 0 0.1"/>  <!-- ตั้ง origin ใหม่ -->
             <geometry>
-                <box size="0.34 0.34 0.725"/>  <!-- size in meter -->
+                <box size="0.34 0.34 0.2"/>  <!-- size in meter -->
             </geometry>
         </collision>
-        <xacro:inertial_box mass="0.5" x="0.34" y="0.34" z="0.725">
-            <origin xyz="0.17 0 0.3625" rpy="0 0 0"/>
+        <xacro:inertial_box mass="0.5" x="0.34" y="0.34" z="0.2">
+            <origin xyz="0.17 0 0.1" rpy="0 0 0"/>
         </xacro:inertial_box>
     </link>
